File: mlx_dev_board.brd (EAGLE design)
At the start: 19 x 12.6 mm, 6 parts, among them U2 MLX90640ESF-BAB-000-TU

Commit message: improvements
Parts:
- removed C3: 10u, resistor:C0805
- added C2: 10u, resistor:C0805
- U1: value MLX90640ESF-BAB-000-TU -> MLX90640
- moved C1 2.29 mm to (4.57, 8.89)
- renumbered U2 to U1
Connections:
- net GND: now also C2.2; no longer C3.2
- net VDD: now also C2.1; no longer C3.1
Changed lines of the file:
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@@
 <layer number="17" name="Pads" color="2" fill="1" visible="yes" active="yes"/>
 <layer number="18" name="Vias" color="2" fill="1" visible="yes" active="yes"/>
-<layer number="19" name="Unrouted" color="6" fill="1" visible="no" active="yes"/>
+<layer number="19" name="Unrouted" color="6" fill="1" visible="yes" active="yes"/>
 <layer number="20" name="Dimension" color="15" fill="1" visible="yes" active="yes"/>
-<layer number="21" name="tPlace" color="7" fill="1" visible="no" active="yes"/>
-<layer number="22" name="bPlace" color="7" fill="1" visible="no" active="yes"/>
-<layer number="23" name="tOrigins" color="15" fill="1" visible="no" active="yes"/>
-<layer number="24" name="bOrigins" color="15" fill="1" visible="no" active="yes"/>
-<layer number="25" name="tNames" color="7" fill="1" visible="no" active="yes"/>
-<layer number="26" name="bNames" color="7" fill="1" visible="no" active="yes"/>
+<layer number="21" name="tPlace" color="7" fill="1" visible="yes" active="yes"/>
+<layer number="22" name="bPlace" color="7" fill="1" visible="yes" active="yes"/>
+<layer number="23" name="tOrigins" color="15" fill="1" visible="yes" active="yes"/>
+<layer number="24" name="bOrigins" color="15" fill="1" visible="yes" active="yes"/>
+<layer number="25" name="tNames" color="7" fill="1" visible="yes" active="yes"/>
+<layer number="26" name="bNames" color="7" fill="1" visible="yes" active="yes"/>
 <layer number="27" name="tValues" color="7" fill="1" visible="no" active="yes"/>
 <layer number="28" name="bValues" color="7" fill="1" visible="no" active="yes"/>
@@
 <layer number="42" name="bRestrict" color="1" fill="10" visible="no" active="yes"/>
 <layer number="43" name="vRestrict" color="2" fill="10" visible="no" active="yes"/>
-<layer number="44" name="Drills" color="7" fill="1" visible="no" active="yes"/>
-<layer number="45" name="Holes" color="7" fill="1" visible="no" active="yes"/>
+<layer number="44" name="Drills" color="7" fill="1" visible="yes" active="yes"/>
+<layer number="45" name="Holes" color="7" fill="1" visible="yes" active="yes"/>
 <layer number="46" name="Milling" color="3" fill="1" visible="no" active="yes"/>
-<layer number="47" name="Measures" color="7" fill="1" visible="no" active="yes"/>
-<layer number="48" name="Document" color="7" fill="1" visible="no" active="yes"/>
-<layer number="49" name="Reference" color="7" fill="1" visible="no" active="yes"/>
+<layer number="47" name="Measures" color="7" fill="1" visible="yes" active="yes"/>
+<layer number="48" name="Document" color="7" fill="1" visible="yes" active="yes"/>
+<layer number="49" name="Reference" color="7" fill="1" visible="yes" active="yes"/>
 <layer number="50" name="dxf" color="7" fill="1" visible="no" active="no"/>
-<layer number="51" name="tDocu" color="7" fill="1" visible="no" active="yes"/>
-<layer number="52" name="bDocu" color="7" fill="1" visible="no" active="yes"/>
+<layer number="51" name="tDocu" color="7" fill="1" visible="yes" active="yes"/>
+<layer number="52" name="bDocu" color="7" fill="1" visible="yes" active="yes"/>
 <layer number="53" name="tGND_GNDA" color="7" fill="1" visible="no" active="no"/>
 <layer number="54" name="bGND_GNDA" color="7" fill="1" visible="no" active="no"/>
@@
 </autorouter>
 <elements>
-<element name="C1" library="resistor" package="C0805" value="100n" x="2.286" y="8.89" rot="R270"/>
-<element name="C3" library="resistor" package="C0805" value="10u" x="4.572" y="8.89" rot="R270"/>
+<element name="C2" library="resistor" package="C0805" value="10u" x="2.286" y="8.89" rot="R270"/>
+<element name="C1" library="resistor" package="C0805" value="100n" x="4.572" y="8.89" rot="R270"/>
 <element name="JP1" library="pinhead" package="1X04" value="CONTROL" x="-0.254" y="6.35" rot="R269.7"/>
 <element name="R1" library="resistor" package="R0805" value="2k" x="12.7" y="10.16" rot="R180"/>
 <element name="R2" library="resistor" package="R0805" value="2k" x="10.668" y="7.112" rot="R90"/>
-<element name="U2" library="MLX90640ESF-BAB-000-TU" package="TO292P945H1165-4" value="MLX90640ESF-BAB-000-TU" x="10.922" y="6.35" rot="R247.9">
+<element name="U1" library="MLX90640ESF-BAB-000-TU" package="TO292P945H1165-4" value="MLX90640" x="10.922" y="6.35" rot="R247.9">
 <attribute name="MF" value="Melexis Technologies NV" x="10.922" y="6.35" size="1.778" layer="27" rot="R247.9" display="off"/>
 <attribute name="DESCRIPTION" value=" Thermal Image Sensor 32H x 24V - TO-39 " x="10.922" y="6.35" size="1.778" layer="27" rot="R247.9" display="off"/>
@@
 <signals>
 <signal name="VDD">
-<contactref element="U2" pad="2"/>
+<contactref element="U1" pad="2"/>
 <contactref element="JP1" pad="1"/>
 <contactref element="R2" pad="2"/>
 <contactref element="R1" pad="2"/>
-<contactref element="C3" pad="1"/>
 <contactref element="C1" pad="1"/>
+<contactref element="C2" pad="1"/>
 <wire x1="-0.23405" y1="10.159946875" x2="1.966053125" y2="10.159946875" width="1.016" layer="1"/>
 <wire x1="1.966053125" y1="10.159946875" x2="2.286" y2="9.84" width="1.016" layer="1"/>
@@
 <signal name="GND">
 <contactref element="JP1" pad="2"/>
-<contactref element="U2" pad="3"/>
-<contactref element="C3" pad="2"/>
+<contactref element="U1" pad="3"/>
 <contactref element="C1" pad="2"/>
+<contactref element="C2" pad="2"/>
 <wire x1="-0.24735" y1="7.61998125" x2="1.96598125" y2="7.61998125" width="1.016" layer="1"/>
 <wire x1="1.96598125" y1="7.61998125" x2="2.286" y2="7.94" width="1.016" layer="1"/>
@@
 </signal>
 <signal name="SDA">
-<contactref element="U2" pad="1"/>
+<contactref element="U1" pad="1"/>
 <contactref element="JP1" pad="4"/>
 <contactref element="R1" pad="1"/>
@@
 </signal>
 <signal name="SCL">
-<contactref element="U2" pad="4"/>
+<contactref element="U1" pad="4"/>
 <contactref element="JP1" pad="3"/>
 <contactref element="R2" pad="1"/>
